File: keyboard-prototype.kicad_pcb (KiCad board)
At the start: 2 copper layers, 77.5 x 61 mm, 18 parts, among them SW1 SW_PUSH, SW2 SW_PUSH, SW3 SW_PUSH, SW4 SW_PUSH, SW5 SW_PUSH, SW6 SW_PUSH, SW7 SW_PUSH, SW8 SW_PUSH, SW9 SW_PUSH

Commit message: Autorouting
Parts:
- added U1: Teensy3.2, prototype:TeensySimple, F.Cu at (152.4, 45.7)
- turned SW3 to 90 degrees
Routing:
- net Net-(D1-Pad1): track 180.9 -> 59.3 mm, vias 1 -> 0
- net Net-(SW3-Pad1): track 130.8 -> 51.2 mm, vias 1 -> 0
- net Net-(SW2-Pad1): track 148.2 -> 70.4 mm, vias 1 -> 0
- net Net-(D4-Pad1): track 120.0 -> 46.6 mm, vias 1 -> 0
- net Net-(D7-Pad1): track 70.2 -> 67.0 mm, vias 1 -> 0
- net Net-(SW1-Pad1): track 91.5 -> 93.0 mm, vias 1 -> 0
- net Net-(D3-Pad2): track 13.3 -> 14.6 mm
Other:
- board size 77.5 x 61 mm -> 88.9 x 61 mm
